Commit message: Demonstrate Gazebo simulation

File: src/ex05_gz_control/description/ros2_control/diffbot.ros2_control.xacro (robot description, xacro)
@@ -1,21 +1,27 @@
 <?xml version="1.0"?>
 <robot xmlns:xacro="http://www.ros.org/wiki/xacro">
-  <xacro:macro name="diffbot_ros2_control">
-    <ros2_control name="DiffBot" type="system">
-        <hardware>
-          <plugin>mock_components/GenericSystem</plugin>
-          <param name="calculate_dynamics">true</param>
-        </hardware>
-      <joint name="wheel_l_joint">
-        <command_interface name="velocity"/>
-        <state_interface name="position"/>
-        <state_interface name="velocity"/>
-      </joint>
-      <joint name="wheel_r_joint">
-        <command_interface name="velocity"/>
-        <state_interface name="position"/>
-        <state_interface name="velocity"/>
-      </joint>
-    </ros2_control>
-  </xacro:macro>
+    <xacro:include filename="diffdrivebot_params.xacro" />
+    <xacro:macro name="diffbot_ros2_control">
+        <ros2_control name="GazeboSystem" type="system">
+            <hardware>
+                <plugin>gz_ros2_control/GazeboSimSystem</plugin>
+            </hardware>
+            <joint name="wheel_l_joint">
+                <command_interface name="velocity">
+                    <param name="min">-10</param>
+                    <param name="max">10</param>
+                </command_interface>
+                <state_interface name="position" />
+                <state_interface name="velocity" />
+            </joint>
+            <joint name="wheel_r_joint">
+                <command_interface name="velocity">
+                    <param name="min">-10</param>
+                    <param name="max">10</param>
+                </command_interface>
+                <state_interface name="position" />
+                <state_interface name="velocity" />
+            </joint>
+        </ros2_control>
+    </xacro:macro>
 </robot>

File: src/ex05_gz_control/description/urdf/diffdrivebot.urdf.xacro (robot description, xacro)
@@ -6,5 +6,8 @@
     <xacro:include filename="diffdrivebot_params.xacro" />
     <xacro:include filename="diffbot.ros2_control.xacro" />
+    <xacro:include filename="diffbot.gazebo.xacro" />
+    <!-- Load ros2 and gazebo plugins -->
     <xacro:diffbot_ros2_control/>
+    <xacro:diffbot_gazebo/>
     <!-- Base link -->
     <link name="base_link" />
@@ -35,8 +38,8 @@
     </link>
     <joint name="wheel_l_joint" type="continuous">
-        <origin xyz="0 ${base_depth/2+0.005} 0" rpy="-${pi/2} 0 0"/>
+        <origin xyz="0 ${base_depth/2+wheel_height+0.005} 0" rpy="${pi/2} 0 0"/>
         <parent link="base_link"/>
         <child link="wheel_l_link"/>
-        <axis xyz="0 0 1"/>
+        <axis xyz="0 0 -1"/>
     </joint>
     <link name="wheel_l_link">
@@ -59,5 +62,5 @@
     </link>
     <joint name="wheel_r_joint" type="continuous">
-        <origin xyz="0 -${base_depth/2+wheel_height+0.005} 0" rpy="${pi/2} 0 0"/>
+        <origin xyz="0 -${base_depth/2+0.005} 0" rpy="${pi/2} 0 0"/>
         <parent link="base_link"/>
         <child link="wheel_r_link"/>

File: src/ex05_gz_control/description/urdf/diffdrivebot_params.xacro (robot description, xacro)
@@ -2,5 +2,5 @@
 <robot xmlns:xacro="http://www.ros.org/wiki/xacro" >
     <!-- Read config YAML -->
-    <xacro:property name="yaml_file" value="$(find ex04_ros2_control)/config/robot_controllers.yaml" />
+    <xacro:property name="yaml_file" value="$(find ex05_gz_control)/config/robot_controllers.yaml" />
     <xacro:property name="dict_base" value="${xacro.load_yaml(yaml_file)}"/>
     <xacro:property name="dict_ctrl" value="${dict_base['diffbot_base_controller']['ros__parameters']}"/>

File: src/ex05_gz_control/description/urdf/materials.xacro (robot description, xacro)
@@ -10,3 +10,24 @@
         <color rgba="1 0 0 1"/>
     </material>
+    <!-- Gazebo colors -->
+    <gazebo reference="chassis_link">
+        <material>Gazebo/Red</material>
+        <mu1>0.2</mu1>
+        <mu2>0.2</mu2>
+    </gazebo>
+    <gazebo reference="wheel_l_link">
+        <material>Gazebo/Black</material>
+        <mu1>0.2</mu1>
+        <mu2>0.2</mu2>
+    </gazebo>
+    <gazebo reference="Wheel_r_link">
+        <material>Gazebo/Black</material>
+        <mu1>0.2</mu1>
+        <mu2>0.2</mu2>
+    </gazebo>
+    <gazebo reference="caster_link">
+        <material>Gazebo/Grey</material>
+        <mu1>0.0000001</mu1>
+        <mu2>0.0000001</mu2>
+    </gazebo>
 </robot>
